File: EthernetBoard.sch (EAGLE design)
At the start: 2 parts

Commit message: Slowly following the examples scattered around the interwebs for the PHY
 Changes to be committed:
	modified:   EthernetBoard.sch
	new file:   EthernetPhy.sch
	new file:   PESD2ETH-AX.lbr
Parts:
- removed BD1: (no value), STM32F4 DISCOVERY:STM32F4-DISCOVERY
- removed U$1: TJA1100, TJA1100:TJA1100
Connections:
- removed net GND: BD1.GND, BD1.GND10, BD1.GND2, BD1.GND3, BD1.GND4, BD1.GND5, BD1.GND6, BD1.GND7, BD1.GND8, BD1.GND9, U$1.GND, U$1.GND2
- removed net VDD: BD1.VDD, BD1.VDD2, U$1.V_DD(IO), U$1.V_DD(IO)2
Changed lines of the file:
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@@
 </classes>
 <parts>
-<part name="BD1" library="STM32F4 DISCOVERY" deviceset="STM32F4-DISCOVERY" device=""/>
-<part name="U$1" library="TJA1100" deviceset="TJA1100" device="" package3d_urn="urn:adsk.eagle:package:11413937/1"/>
 </parts>
 <sheets>
@@
 </plain>
 <instances>
-<instance part="BD1" gate="G$1" x="698.5" y="139.7" smashed="yes">
-<attribute name="NAME" x="701.04" y="172.72" size="1.27" layer="94"/>
-</instance>
-<instance part="U$1" gate="G$1" x="601.98" y="142.24" smashed="yes"/>
 </instances>
 <busses>
 </busses>
 <nets>
-<net name="VDD" class="0">
-<segment>
-<pinref part="U$1" gate="G$1" pin="V_DD(IO)2"/>
-<wire x1="607.06" y1="154.94" x2="642.62" y2="154.94" width="0.1524" layer="91"/>
-<wire x1="642.62" y1="154.94" x2="642.62" y2="134.62" width="0.1524" layer="91"/>
-<pinref part="U$1" gate="G$1" pin="V_DD(IO)"/>
-<wire x1="642.62" y1="134.62" x2="607.06" y2="134.62" width="0.1524" layer="91"/>
-</segment>
-<segment>
-<pinref part="BD1" gate="G$1" pin="VDD"/>
-<wire x1="693.42" y1="165.1" x2="675.64" y2="165.1" width="0.1524" layer="91"/>
-<wire x1="675.64" y1="165.1" x2="675.64" y2="185.42" width="0.1524" layer="91"/>
-<wire x1="675.64" y1="185.42" x2="739.14" y2="185.42" width="0.1524" layer="91"/>
-<wire x1="739.14" y1="185.42" x2="739.14" y2="165.1" width="0.1524" layer="91"/>
-<pinref part="BD1" gate="G$1" pin="VDD2"/>
-<wire x1="739.14" y1="165.1" x2="723.9" y2="165.1" width="0.1524" layer="91"/>
-</segment>
-</net>
-<net name="GND" class="0">
-<segment>
-<pinref part="U$1" gate="G$1" pin="GND"/>
-<wire x1="594.36" y1="129.54" x2="594.36" y2="83.82" width="0.1524" layer="91"/>
-<wire x1="594.36" y1="83.82" x2="652.78" y2="83.82" width="0.1524" layer="91"/>
-<wire x1="652.78" y1="83.82" x2="652.78" y2="152.4" width="0.1524" layer="91"/>
-<pinref part="U$1" gate="G$1" pin="GND2"/>
-<wire x1="652.78" y1="152.4" x2="607.06" y2="152.4" width="0.1524" layer="91"/>
-</segment>
-<segment>
-<pinref part="BD1" gate="G$1" pin="GND5"/>
-<wire x1="693.42" y1="106.68" x2="693.42" y2="96.52" width="0.1524" layer="91"/>
-<wire x1="693.42" y1="96.52" x2="723.9" y2="96.52" width="0.1524" layer="91"/>
-<pinref part="BD1" gate="G$1" pin="GND6"/>
-<wire x1="723.9" y1="96.52" x2="723.9" y2="106.68" width="0.1524" layer="91"/>
-<pinref part="BD1" gate="G$1" pin="GND4"/>
-<wire x1="693.42" y1="139.7" x2="688.34" y2="139.7" width="0.1524" layer="91"/>
-<wire x1="688.34" y1="139.7" x2="688.34" y2="96.52" width="0.1524" layer="91"/>
-<wire x1="688.34" y1="96.52" x2="693.42" y2="96.52" width="0.1524" layer="91"/>
-<junction x="693.42" y="96.52"/>
-<pinref part="BD1" gate="G$1" pin="GND3"/>
-<wire x1="693.42" y1="162.56" x2="688.34" y2="162.56" width="0.1524" layer="91"/>
-<wire x1="688.34" y1="162.56" x2="688.34" y2="139.7" width="0.1524" layer="91"/>
-<junction x="688.34" y="139.7"/>
-<pinref part="BD1" gate="G$1" pin="GND"/>
-<wire x1="693.42" y1="167.64" x2="688.34" y2="167.64" width="0.1524" layer="91"/>
-<wire x1="688.34" y1="167.64" x2="688.34" y2="162.56" width="0.1524" layer="91"/>
-<junction x="688.34" y="162.56"/>
-<pinref part="BD1" gate="G$1" pin="GND2"/>
-<wire x1="723.9" y1="167.64" x2="728.98" y2="167.64" width="0.1524" layer="91"/>
-<wire x1="728.98" y1="167.64" x2="728.98" y2="175.26" width="0.1524" layer="91"/>
-<wire x1="728.98" y1="175.26" x2="688.34" y2="175.26" width="0.1524" layer="91"/>
-<wire x1="688.34" y1="175.26" x2="688.34" y2="167.64" width="0.1524" layer="91"/>
-<junction x="688.34" y="167.64"/>
-<pinref part="BD1" gate="G$1" pin="GND7"/>
-<wire x1="751.84" y1="167.64" x2="728.98" y2="167.64" width="0.1524" layer="91"/>
-<junction x="728.98" y="167.64"/>
-<pinref part="BD1" gate="G$1" pin="GND8"/>
-<wire x1="782.32" y1="167.64" x2="782.32" y2="175.26" width="0.1524" layer="91"/>
-<wire x1="782.32" y1="175.26" x2="728.98" y2="175.26" width="0.1524" layer="91"/>
-<junction x="728.98" y="175.26"/>
-<pinref part="BD1" gate="G$1" pin="GND9"/>
-<wire x1="751.84" y1="106.68" x2="749.3" y2="106.68" width="0.1524" layer="91"/>
-<wire x1="749.3" y1="106.68" x2="749.3" y2="96.52" width="0.1524" layer="91"/>
-<wire x1="749.3" y1="96.52" x2="723.9" y2="96.52" width="0.1524" layer="91"/>
-<junction x="723.9" y="96.52"/>
-<pinref part="BD1" gate="G$1" pin="GND10"/>
-<wire x1="782.32" y1="106.68" x2="784.86" y2="106.68" width="0.1524" layer="91"/>
-<wire x1="784.86" y1="106.68" x2="784.86" y2="96.52" width="0.1524" layer="91"/>
-<wire x1="784.86" y1="96.52" x2="749.3" y2="96.52" width="0.1524" layer="91"/>
-<junction x="749.3" y="96.52"/>
-</segment>
-</net>
 </nets>
 </sheet>
@@
 </schematic>
 </drawing>
-<compatibility>
-<note version="6.3" minversion="6.2.2" severity="warning">
-Since Version 6.2.2 text objects can contain more than one line,
-which will not be processed correctly with this version.
-</note>
-<note version="8.3" severity="warning">
-Since Version 8.3, EAGLE supports URNs for individual library
-assets (packages, symbols, and devices). The URNs of those assets
-will not be understood (or retained) with this version.
-</note>
-<note version="8.3" severity="warning">
-Since Version 8.3, EAGLE supports the association of 3D packages
-with devices in libraries, schematics, and board files. Those 3D
-packages will not be understood (or retained) with this version.
-</note>
-</compatibility>
 </eagle>
